File: MAQUINA_DE_BRAILLE/DRIVERS.kicad_sch (KiCad schematic)
At the start: 26 parts, among them J1 Screw_Terminal_01x04, J2 Screw_Terminal_01x04, U2 DRV8825PWPR, U3 DRV8825PWPR

Commit message: last update
Parts:
- removed C16, C20: 100uf/16v, Capacitor_SMD:C_0805_2012Metric_Pad1.18x1.45mm_HandSolder, symbol Device:C_Polarized
- added C16, C20: 100uF/16v, EEETC1C101XV:CAP_EEETC1C101XV, symbol EEETC1C101XV:EEETC1C101XV
Connections:
- net GND: now also C16.2, C20.2
- net VCC: now also C16.1, C20.1

Commit message: LAST UPDATE
Parts:
- removed C16, C20: 100uF/16v, EEETC1C101XV:CAP_EEETC1C101XV, symbol EEETC1C101XV:EEETC1C101XV
- added C16, C20: 100uF/35V, 865080545012:CAP_WCAP-ASLI_06p3X07p7_WRE, symbol 865080545012:865080545012
Connections:
- net GND: now also C16.2, C20.2
- net VCC: now also C16.1, C20.1
