File: MAQUINA_DE_BRAILLE/ESP32.kicad_sch (KiCad schematic)
At the start: 18 parts, among them J4 USB_C_Receptacle_USB2.0_16P, J5 Screw_Terminal_01x03, J6 Screw_Terminal_01x03, J7 Screw_Terminal_01x02, Q1 IRLZ44NSTRLPBF, SW1 TS-1088-AR02016, SW2 TS-1088-AR02016, U1 ESP32-S3-WROOM-1-N16

Commit message: tuki
Parts:
- added J8: Screw_Terminal_01x16, TerminalBlock:TerminalBlock_Xinya_XY308-2.54-16P_1x16_P2.54mm_Horizontal, symbol Connector:Screw_Terminal_01x16
Connections:
- net MODE0_TO_ESP32: now also U1.22 (IO14); no longer U1.20 (IO12)
- net MODE2_TO_ESP32: now also U1.20 (IO12); no longer U1.22 (IO14)
- net IO21: now reaches U1.23 (IO21)
- net IO21: now also J8.16 (Pin_16)
- net IO47: now reaches U1.24 (IO47)
- net IO47: now also J8.15 (Pin_15)
- net IO48: now reaches U1.25 (IO48)
- net IO48: now also J8.14 (Pin_14)
- net IO45: now reaches U1.26 (IO45)
- net IO45: now also J8.13 (Pin_13)
- net IO35: now reaches U1.28 (IO35)
- net IO35: now also J8.12 (Pin_12)
- net IO36: now reaches U1.29 (IO36)
- net IO36: now also J8.11 (Pin_11)
- net IO37: now reaches U1.30 (IO37)
- net IO37: now also J8.10 (Pin_10)
- net IO38: now reaches U1.31 (IO38)
- net IO38: now also J8.9 (Pin_9)
- net IO39: now reaches U1.32 (IO39)
- net IO39: now also J8.8 (Pin_8)
- net IO40: now reaches U1.33 (IO40)
- net IO40: now also J8.7 (Pin_7)
- net IO41: now reaches U1.34 (IO41)
- net IO41: now also J8.6 (Pin_6)
- net IO42: now reaches U1.35 (IO42)
- net IO42: now also J8.5 (Pin_5)
- net RXDO: now reaches U1.36 (RXD0)
- net RXDO: now also J8.4 (Pin_4)
- net TXDO: now reaches U1.37 (TXD0)
- net TXDO: now also J8.3 (Pin_3)
- net IO2: now reaches U1.38 (IO2)
- net IO2: now also J8.2 (Pin_2)
- net IO1: now reaches U1.39 (IO1)
- net IO1: now also J8.1 (Pin_1)
- no-connect marks 21 -> 5

Commit message: fabri puto
Parts:
- added NT1: NetTie_2, NetTie:NetTie-2_SMD_Pad2.0mm, symbol Device:NetTie_2
Connections:
- net GND: now also NT1.1
- net GNDD: now also NT1.2
Changed lines of the file:
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@@
+	)
+	(symbol
+		(lib_id "Device:NetTie_2")
+		(at 129.032 41.91 0)
+		(unit 1)
+		(exclude_from_sim no)
+		(in_bom no)
+		(on_board yes)
+		(dnp no)
+		(fields_autoplaced yes)
+		(property "Reference" "NT1"
+			(at 129.032 36.83 0)
+			(effects
+				(font
+					(size 1.27 1.27)
+				)
+			)
+		)
+		(property "Value" "NetTie_2"
+			(at 129.032 39.37 0)
+			(effects
+				(font
+					(size 1.27 1.27)
+				)
+			)
+		)
+		(property "Footprint" "NetTie:NetTie-2_SMD_Pad2.0mm"
+			(at 129.032 41.91 0)
+			(effects
+				(font
+					(size 1.27 1.27)
+				)
+				(hide yes)
+			)
+		)
+		(property "Datasheet" "~"
+			(at 129.032 41.91 0)
+			(effects
+				(font
+					(size 1.27 1.27)
+				)
+				(hide yes)
+			)
+		)
+		(property "Description" "Net tie, 2 pins"
+			(at 129.032 41.91 0)
+			(effects
+				(font
+					(size 1.27 1.27)
+				)
+				(hide yes)
+			)
+		)
+		(pin "2"
+		)
+		(pin "1"
+		)
+		(instances
+			(project ""
+				(path "/9a6fa5b9-6251-4c76-8504-ded4de8e2fcc/099b3b04-aaec-4710-a9d4-459b316d99df"
+					(reference "NT1")
+					(unit 1)
+				)
+			)
+		)
 	)
 	(symbol
@@
 	)
 	(symbol
+		(lib_id "power:GNDD")
+		(at 131.572 41.91 0)
+		(unit 1)
+		(exclude_from_sim no)
+		(in_bom yes)
+		(on_board yes)
+		(dnp no)
+		(fields_autoplaced yes)
+		(property "Reference" "#PWR018"
+			(at 131.572 48.26 0)
+			(effects
+				(font
+					(size 1.27 1.27)
+				)
+				(hide yes)
+			)
+		)
+		(property "Value" "GNDD"
+			(at 131.572 45.72 0)
+			(effects
+				(font
+					(size 1.27 1.27)
+				)
+			)
+		)
+		(property "Footprint" ""
+			(at 131.572 41.91 0)
+			(effects
+				(font
+					(size 1.27 1.27)
+				)
+				(hide yes)
+			)
+		)
+		(property "Datasheet" ""
+			(at 131.572 41.91 0)
+			(effects
+				(font
+					(size 1.27 1.27)
+				)
+				(hide yes)
+			)
+		)
+		(property "Description" "Power symbol creates a global label with name \"GNDD\" , digital ground"
+			(at 131.572 41.91 0)
+			(effects
+				(font
+					(size 1.27 1.27)
+				)
+				(hide yes)
+			)
+		)
+		(pin "1"
+		)
+		(instances
+			(project ""
+				(path "/9a6fa5b9-6251-4c76-8504-ded4de8e2fcc/099b3b04-aaec-4710-a9d4-459b316d99df"
+					(reference "#PWR018")
+					(unit 1)
+				)
+			)
+		)
+	)
+	(symbol
 		(lib_id "Connector:Screw_Terminal_01x03")
 		(at 58.674 150.368 180)
@@
 					(unit 1)
 				)
+			)
+		)
+	)
+	(symbol
+		(lib_id "power:GND")
+		(at 126.492 41.91 0)
+		(unit 1)
+		(exclude_from_sim no)
+		(in_bom yes)
+		(on_board yes)
+		(dnp no)
+		(fields_autoplaced yes)
+		(property "Reference" "#PWR017"
+			(at 126.492 48.26 0)
+			(effects
+				(font
+					(size 1.27 1.27)
+				)
+				(hide yes)
+			)
+		)
+		(property "Value" "GND"
+			(at 126.492 46.99 0)
+			(effects
+				(font
+					(size 1.27 1.27)
+				)
+			)
+		)
+		(property "Footprint" ""
+			(at 126.492 41.91 0)
+			(effects
+				(font
+					(size 1.27 1.27)
+				)
+				(hide yes)
+			)
+		)
+		(property "Datasheet" ""
+			(at 126.492 41.91 0)
+			(effects
+				(font
+					(size 1.27 1.27)
+				)
+				(hide yes)
+			)
+		)
+		(property "Description" "Power symbol creates a global label with name \"GND\" , ground"
+			(at 126.492 41.91 0)
+			(effects
+				(font
+					(size 1.27 1.27)
+				)
+				(hide yes)
+			)
+		)
+		(pin "1"
+		)
+		(instances
+			(project ""
+				(path "/9a6fa5b9-6251-4c76-8504-ded4de8e2fcc/099b3b04-aaec-4710-a9d4-459b316d99df"
+					(reference "#PWR017")
+					(unit 1)
+				)
