File: MAQUINA_DE_BRAILLE/MAQUINA_DE_BRAILLE.kicad_pcb (KiCad board)
At the start: 4 copper layers, 80.2 x 81.1 mm, 69 parts, among them J1 Screw_Terminal_01x04, J2 Screw_Terminal_01x04, J3 Screw_Terminal_01x02, J4 USB_C_Receptacle_USB2.0_16P, J5 Screw_Terminal_01x03, J6 Screw_Terminal_01x03, J7 Screw_Terminal_01x02, J8 Screw_Terminal_01x16, Q1 IRLZ44NSTRLPBF, SW1 TS-1088-AR02016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

Commit message: Update MAQUINA_DE_BRAILLE.kicad_pcb
Routing:
- net GND: track 50.2 -> 49.3 mm
Changed lines of the file:
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@@
+	)
+	(segment
+		(start 146.44 106.959)
+		(end 146.44 104.37)
+		(width 0.4)
+		(layer "F.Cu")
+		(net 8)
 	)
 	(segment
@@
 	)
 	(segment
-		(start 146.44 106.959)
-		(end 146.44 103.46)
-		(width 0.4)
-		(layer "F.Cu")
-		(net 8)
-	)
-	(segment
 		(start 133.1718 70.2318)
 		(end 133.17 70.23)
@@
 	)
 	(via
-		(at 146.44 103.46)
-		(size 0.7)
-		(drill 0.3)
+		(at 146.44 104.37)
+		(size 0.7)
+		(drill 0.3)

Commit message: last update
Parts:
- C16, C20: value 100uf/16v -> 100uF/16v; footprint Capacitor_SMD:C_0805_2012Metric_Pad1.18x1.45mm_HandSolder -> EEETC1C101XV:CAP_EEETC1C101XV
- moved C16 24.4 mm to (112.0, 68.7), turned to 90 degrees
- moved C20 21.2 mm to (112.3, 91.1), turned to 90 degrees
- moved C19 2.59 mm to (116.8, 70.4)
- moved C15 2.50 mm to (117.6, 92.5)
Routing:
- net VCC: track 259.4 -> 266.1 mm
- net GND: track 49.3 -> 51.1 mm
Other:
- board size 80.2 x 81.1 mm -> 84.5 x 81.1 mm

Commit message: LAST UPDATE
Parts:
- C16, C20: value 100uF/16v -> 100uF/35V; footprint EEETC1C101XV:CAP_EEETC1C101XV -> 865080545012:CAP_WCAP-ASLI_06p3X07p7_WRE
- C5, C6: value 4.7uf -> 10uF/10v; footprint Capacitor_SMD:C_0805_2012Metric_Pad1.18x1.45mm_HandSolder -> 293D106X9010A2TE3:CAP_293D-A_VSS
- LDO1: value ADP122AUJZ-3.3-R7 -> LM1117MPX-33NOPB; footprint ADP122AUJZ_3_3_R7:UJ_5_ADI -> LM1117:SOT223-318H_OSI
- MOSFET1: value AO3401A -> DMP3130L-7; footprint AO3401A:SOT-23-3L_AOS -> DMP3130L-7:SOT-23_DMP3130L_DIO
- moved C20 26.2 mm to (111.3, 64.9)
- moved C16 21.1 mm to (112.1, 89.8)
- moved R24 8.22 mm to (150.5, 103.0), turned to 180 degrees
- moved R5 7.08 mm to (167.5, 96.2), turned to -90 degrees
- moved J4 5.87 mm to (112.3, 52.0)
- moved LDO1 5.79 mm to (159.1, 91.1), turned to 90 degrees
- moved D2 5.69 mm to (167.4, 92.2), turned to 90 degrees
- moved C19 3.62 mm to (117.0, 66.8)
- moved R20 3.57 mm to (122.0, 77.1)
- moved R21 3.57 mm to (122.0, 74.9)
- moved C21 3.57 mm to (121.6, 66.7)
- moved C22 3.57 mm to (124.1, 66.7)
- moved C24 3.57 mm to (137.3, 77.0)
- moved J1 3.57 mm to (115.0, 79.9)
- moved R15 3.57 mm to (119.2, 66.7)
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Connections:
- LDO1 pad 1: MOSFET_TO_LDO -> GND
- LDO1 pad 2: GND -> VCC_3V3
Routing:
- net Net-(U1-IO15): track 46.4 -> 59.0 mm
- net VCC: track 266.1 -> 277.1 mm
- net Net-(Q1-G): track 11.3 -> 3.95 mm
- net Net-(J4-CC1): track 7.24 -> 13.8 mm
- net USB_TO_MOSFET: track 65.3 -> 71.4 mm
- net Net-(J4-CC2): track 6.67 -> 12.6 mm
- net USB_D+: track 43.7 -> 49.7 mm
- net USB_D-: track 43.8 -> 49.7 mm
- net GNDD: track 45.4 -> 49.5 mm, vias 17 -> 19
- net VCC_3V3: track 13.8 -> 17.7 mm, vias 5 -> 3
- net MODE2_TO_ESP32: track 71.6 -> 75.4 mm
- net BUCK_TO_MOSFET: track 36.4 -> 39.5 mm
- net DRIVER_X_nFAULT_TO_ESP32: track 38.7 -> 41.1 mm
- net DRIVER_X_nENBL_TO_ESP32: track 39.1 -> 40.8 mm
- net MODE1_TO_ESP32: track 75.5 -> 77.1 mm
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
Commit message: fabri puto
Parts:
- added NT1: NetTie_2, NetTie:NetTie-2_SMD_Pad2.0mm, F.Cu at (174.5, 119.5)
Routing:
- net GND: track 50.9 -> 55.6 mm, vias 33 -> 35
- net GNDD: track 49.5 -> 51.3 mm, vias 19 -> 20
- net VCC: track 277.1 -> 278.2 mm
Changed lines of the file:
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@@
 	(layers
 		(0 "F.Cu" signal)
-		(4 "In1.Cu" power "GND")
-		(6 "In2.Cu" signal)
-		(2 "B.Cu" signal)
+		(4 "In1.Cu" power "GNDD")
+		(6 "In2.Cu" power "GND")
+		(2 "B.Cu" power)
 		(9 "F.Adhes" user "F.Adhesive")
 		(11 "B.Adhes" user "B.Adhesive")
@@
 		(embedded_fonts no)
 	)
+	(footprint "NetTie:NetTie-2_SMD_Pad2.0mm"
+		(layer "F.Cu")
+		(at 174.498 119.5324 90)
+		(descr "Net tie, 2 pin, 2.0mm square SMD pads")
+		(tags "net tie")
+		(property "Reference" "NT1"
+			(at 0 -2 90)
+			(layer "F.SilkS")
+			(hide yes)
+			(effects
+				(font
+					(size 1 1)
+					(thickness 0.15)
+				)
+			)
+		)
+		(property "Value" "NetTie_2"
+			(at 0 2 90)
+			(layer "F.Fab")
+			(hide yes)
+			(effects
+				(font
+					(size 1 1)
+					(thickness 0.15)
+				)
+			)
+		)
+		(property "Datasheet" "~"
+			(at 0 0 90)
+			(unlocked yes)
+			(layer "F.Fab")
+			(hide yes)
+			(effects
+				(font
+					(size 1.27 1.27)
+					(thickness 0.15)
+				)
+			)
+		)
+		(property "Description" "Net tie, 2 pins"
+			(at 0 0 90)
+			(unlocked yes)
+			(layer "F.Fab")
+			(hide yes)
+			(effects
+				(font
+					(size 1.27 1.27)
+					(thickness 0.15)
+				)
+			)
+		)
+		(property ki_fp_filters "Net*Tie*")
+		(sheetname "/ESP32/")
+		(sheetfile "ESP32.kicad_sch")
+		(attr exclude_from_pos_files exclude_from_bom allow_missing_courtyard)
+		(net_tie_pad_groups "1, 2")
+		(fp_poly
+			(pts
+				(xy -2 -1) (xy 2 -1) (xy 2 1) (xy -2 1)
+			)
+			(stroke
+				(width 0)
+				(type solid)
+			)
+			(fill yes)
+			(layer "F.Cu")
+		)
+		(pad "1" smd circle
+			(at -2 0 90)
+			(size 2 2)
+			(layers "F.Cu")
+			(net 8 "GND")
+			(pinfunction "1")
+			(pintype "passive")
+		)
+		(pad "2" smd circle
+			(at 2 0 90)
+			(size 2 2)
+			(layers "F.Cu")
+			(net 86 "GNDD")
+			(pinfunction "2")
+			(pintype "passive")
+		)
+		(embedded_fonts no)
+	)
 	(footprint "Resistor_SMD:R_0805_2012Metric_Pad1.20x1.40mm_HandSolder"
 		(layer "F.Cu")
@@
 	)
 	(via
-		(at 175.65 113.64)
+		(at 173.0498 113.64)
 		(size 0.7)
 		(drill 0.3)
@@
 	)
 	(segment
-		(start 118.4425 119.105)
-		(end 122.6475 123.31)
+		(start 175.65 113.64)
+		(end 175.66 113.65)
 		(width 0.7)
 		(layer "B.Cu")
@@
 	)
 	(segment
-		(start 175.66 113.65)
-		(end 175.65 113.64)
+		(start 118.4425 119.105)
+		(end 122.6475 123.31)
 		(width 0.7)
 		(layer "B.Cu")
@@
 	)
 	(segment
-		(start 183.3 113.65)
-		(end 175.66 113.65)
+		(start 173.0498 113.64)
+		(end 175.65 113.64)
+		(width 0.7)
+		(layer "B.Cu")
+		(net 7)
+	)
+	(segment
+		(start 175.66 113.65)
+		(end 183.3 113.65)
 		(width 0.7)
 		(layer "B.Cu")
@@
 	)
 	(segment
+		(start 169.37 78.4)
+		(end 150.64 78.4)
+		(width 0.7)
+		(layer "In2.Cu")
+		(net 7)
+	)
+	(segment
 		(start 123.68 89.66)
 		(end 123.401 89.381)
@@
 	)
 	(segment
-		(start 134.0748 61.8348)
-		(end 137.63 65.39)
+		(start 175.65 84.68)
+		(end 169.37 78.4)
 		(width 0.7)
 		(layer "In2.Cu")
@@
 	)
 	(segment
-		(start 175.65 84.68)
-		(end 175.65 113.64)
-		(width 0.7)
-		(layer "In2.Cu")
-		(net 7)
-	)
-	(segment
-		(start 137.63 65.39)
-		(end 150.64 78.4)
+		(start 150.64 78.4)
+		(end 134.0748 61.8348)
 		(width 0.7)
 		(layer "In2.Cu")
@@
 	)
 	(segment
-		(start 165.98 123.31)
-		(end 175.65 113.64)
+		(start 134.0748 61.8348)
+		(end 124.831 61.8348)
 		(width 0.7)
 		(layer "In2.Cu")
@@
 	)
 	(segment
-		(start 169.37 78.4)
-		(end 175.65 84.68)
+		(start 163.3798 123.31)
+		(end 160.77 123.31)
 		(width 0.7)
 		(layer "In2.Cu")
@@
 	)
 	(segment
-		(start 122.681 63.9848)
-		(end 124.831 61.8348)
+		(start 124.831 61.8348)
+		(end 122.681 63.9848)
 		(width 0.7)
 		(layer "In2.Cu")
@@
 	)
 	(segment
-		(start 150.64 78.4)
-		(end 169.37 78.4)
+		(start 173.0498 113.64)
+		(end 163.3798 123.31)
+		(width 0.7)
+		(layer "In2.Cu")
+		(net 7)
+	)
+	(segment
+		(start 173.0498 113.64)
+		(end 175.65 111.0398)
 		(width 0.7)
 		(layer "In2.Cu")
@@
 	)
 	(segment
-		(start 160.77 123.31)
-		(end 165.98 123.31)
+		(start 175.65 111.0398)
+		(end 175.65 84.68)
 		(width 0.7)
 		(layer "In2.Cu")
@@
 	)
 	(segment
-		(start 124.831 61.8348)
-		(end 134.0748 61.8348)
-		(width 0.7)
-		(layer "In2.Cu")
-		(net 7)
-	)
-	(segment
 		(start 123.401 77.5948)
 		(end 125.401 75.5948)
@@
 	)
 	(segment
+		(start 174.498 123.2662)
+		(end 174.4726 123.2916)
+		(width 0.4)
+		(layer "F.Cu")
+		(net 8)
+	)
+	(segment
+		(start 174.498 121.5324)
+		(end 174.498 123.2662)
+		(width 0.4)
+		(layer "F.Cu")
+		(net 8)
+	)
+	(segment
 		(start 146.44 106.959)
 		(end 146.44 104.37)
@@
 	)
 	(via
+		(at 180.34 118.745)
+		(size 0.7)
+		(drill 0.3)
+		(layers "F.Cu" "B.Cu")
+		(net 8)
+	)
+	(via
 		(at 164.07 114.69)
 		(size 0.7)
@@
 	)
 	(via
+		(at 174.4726 123.2916)
+		(size 0.7)
+		(drill 0.3)
+		(layers "F.Cu" "B.Cu")
+		(net 8)
+	)
+	(via
 		(at 164.11 116.75)
 		(size 0.7)
@@
 	)
 	(segment
+		(start 183.3 118.73)
+		(end 180.355 118.73)
+		(width 0.4)
+		(layer "B.Cu")
+		(net 8)
+	)
+	(segment
+		(start 180.355 118.73)
+		(end 180.34 118.745)
+		(width 0.4)
+		(layer "B.Cu")
+		(net 8)
+	)
+	(segment
 		(start 164.372578 90.763324)
 		(end 164.9464 91.337146)
@@
 	)
 	(segment
+		(start 174.498 117.5324)
+		(end 174.498 115.7224)
+		(width 0.4)
+		(layer "F.Cu")
+		(net 86)
+	)
+	(segment
 		(start 130.29 54.24)
 		(end 132.17 54.24)
@@
 		(net 86)
 	)
+	(via
+		(at 174.498 115.7224)
+		(size 0.7)
+		(drill 0.3)
+		(layers "F.Cu" "B.Cu")
+		(net 86)
+	)
