File: MAQUINA_DE_BRAILLE/MAQUINA_DE_BRAILLE.kicad_pcb (KiCad board)
At the start: 4 copper layers, 84.5 x 81.1 mm, 70 parts, among them J1 Screw_Terminal_01x04, J2 Screw_Terminal_01x04, J3 Screw_Terminal_01x02, J4 USB_C_Receptacle_USB2.0_16P, J5 Screw_Terminal_01x03, J6 Screw_Terminal_01x03, J7 Screw_Terminal_01x02, J8 Screw_Terminal_01x16, Q1 IRLZ44NSTRLPBF, SW1 TS-1088-AR02016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

Commit message: last update
Parts:
- moved J4 1.91 mm to (110.4, 52.1)
Routing:
- net USB_TO_MOSFET: track 71.4 -> 73.6 mm
- net USB_D-: track 49.7 -> 51.8 mm
- net Net-(J4-CC2): track 12.6 -> 14.5 mm
- net USB_D+: track 49.7 -> 51.6 mm
- net Net-(J4-CC1): track 13.8 -> 15.2 mm
