File: MAQUINA_DE_BRAILLE_PCB/MAQUINA_DE_BRAILLE.kicad_pcb (KiCad board)
At the start: 4 copper layers, 84.5 x 81.1 mm, 70 parts, among them J1 Screw_Terminal_01x04, J2 Screw_Terminal_01x04, J3 Screw_Terminal_01x02, J4 USB_C_Receptacle_USB2.0_16P, J5 Screw_Terminal_01x03, J6 Screw_Terminal_01x03, J7 Screw_Terminal_01x02, J8 Screw_Terminal_01x16, Q1 IRLZ44NSTRLPBF, SW1 TS-1088-AR02016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

Commit message: last update
Parts:
- C5, C6: footprint 293D106X9010A2TE3:CAP_293D-A_VSS -> 293D106X9010B2TE3:CAP_293D_B_VIS
- moved C20 18.9 mm to (130.1, 63.4), turned to 0 degrees
- moved C16 18.3 mm to (130.4, 89.0), turned to 0 degrees
- moved LDO1 1.64 mm to (157.6, 91.8)
- moved C5 1.31 mm to (164.6, 89.0)
- moved C6 1.11 mm to (164.2, 93.5)
- moved R5 1.09 mm to (167.3, 97.2)
- moved D2 1.09 mm to (167.2, 93.3)
Routing:
- net BOOT: track 54.8 -> 42.3 mm
- net VCC: track 278.2 -> 269.9 mm
- net BUCK_TO_MOSFET: track 39.5 -> 37.3 mm
- net IO45: track 42.1 -> 43.9 mm, vias 2 -> 1
- net MOSFET_TO_LDO: track 11.3 -> 13.1 mm
- net VCC_3V3: track 17.7 -> 19.1 mm
- net IO48: track 45.1 -> 46.5 mm, vias 2 -> 1
- net IO40: track 35.8 -> 36.9 mm, vias 2 -> 1
- net GND: track 55.6 -> 56.6 mm, vias 35 -> 69
- net IO47: track 48.1 -> 48.9 mm, vias 2 -> 1
- net IO39: track 37.0 -> 37.7 mm, vias 2 -> 1
- net IO41: track 34.6 -> 35.3 mm, vias 2 -> 1
- net IO36: track 40.9 -> 40.4 mm, vias 2 -> 1
- net IO37: track 39.7 -> 39.4 mm, vias 2 -> 1
- net IO21: vias 2 -> 1
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