File: MAQUINA_DE_BRAILLE_PCB/MAQUINA_DE_BRAILLE.kicad_pcb (KiCad board)
At the start: 4 copper layers, 84.5 x 81.1 mm, 70 parts, among them J1 Screw_Terminal_01x04, J2 Screw_Terminal_01x04, J3 Screw_Terminal_01x02, J4 USB_C_Receptacle_USB2.0_16P, J5 Screw_Terminal_01x03, J6 Screw_Terminal_01x03, J7 Screw_Terminal_01x02, J8 Screw_Terminal_01x16, Q1 IRLZ44NSTRLPBF, SW1 TS-1088-AR02016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

Commit message: last update
Parts:
- removed SW1, SW2: TS-1088-AR02016, TS-1088-AR02016:SW_TS-1088_XNP
- added BOOT: 434123025816, SW434123025816:434123025816, F.Cu at (147.4, 49.7)
- added C25: 0.1uf, Capacitor_SMD:C_0805_2012Metric_Pad1.18x1.45mm_HandSolder, F.Cu at (114.7, 66.8)
- added C26: 0.1uf, Capacitor_SMD:C_0805_2012Metric_Pad1.18x1.45mm_HandSolder, F.Cu at (115.6, 92.4)
- added EN: 434123025816, SW434123025816:434123025816, F.Cu at (147.4, 56.4)
- C13: value 0.1uf -> 1nf
- C14: value 6.8uf -> 6.8nf
- R16, R17: value 0.1 -> 0.2
- moved R4 7.13 mm to (155.2, 56.2)
- moved C4 0.81 mm to (155.2, 58.5)
- moved R7 0.25 mm to (157.3, 106.2)
- moved C13 0.24 mm to (158.3, 111.3)
- moved R10 0.20 mm to (165.6, 110.6)
- moved C10 0.16 mm to (162.8, 108.1)
- moved C9 0.13 mm to (165.8, 113.2)
- moved C11 0.11 mm to (162.8, 105.8)
- moved C14 0.10 mm to (159.7, 106.5)
- moved R9 0.08 mm to (161.6, 119.0)
Routing:
- net GNDD: track 51.3 -> 25.4 mm, vias 20 -> 21
- net EN: track 13.3 -> 21.5 mm
- net BOOT: track 42.3 -> 37.4 mm
- net VCC: track 269.9 -> 274.5 mm
- net Net-(R4-Pad1): track 3.82 -> 7.89 mm
- net GND: track 56.6 -> 59.6 mm, vias 69 -> 71
- net Net-(U3-AVREF): track 9.11 -> 8.24 mm
- net VCC_3V3: track 19.1 -> 18.4 mm

Commit message: a
Parts:
- added G***: LOGO, FIUNA_LOGO:FIUNA_LOGO, F.Cu at (148.8, 119.4)
- moved Q1 8.21 mm to (148.8, 106.8)
- moved R24 8.21 mm to (150.3, 94.8)
Routing:
- net Net-(U1-IO15): track 59.0 -> 50.9 mm
- net Net-(J7-Pin_1): track 34.9 -> 33.1 mm

Commit message: a
Parts:
- added H1: MountingHole_Pad, MountingHole:MountingHole_3mm_Pad_Via, F.Cu at (110.6, 48.2)
- added H2: MountingHole_Pad, MountingHole:MountingHole_3mm_Pad_Via, F.Cu at (194.8, 48.2)
- added H3: MountingHole_Pad, MountingHole:MountingHole_3mm_Pad_Via, F.Cu at (110.7, 125.8)
- added H4: MountingHole_Pad, MountingHole:MountingHole_3mm_Pad_Via, F.Cu at (194.8, 125.9)
- moved G*** 11.3 mm to (138.0, 122.6)
- moved R2 9.55 mm to (122.0, 54.4)
- moved R3 8.72 mm to (122.1, 59.1)
- moved J4 5.73 mm to (110.4, 57.8)
- moved J7 3.12 mm to (116.9, 111.3)
- moved CR1 3.12 mm to (129.1, 113.8)
Routing:
- net Net-(J4-CC2): track 14.5 -> 7.16 mm
- net Net-(J4-CC1): track 15.2 -> 7.85 mm
- net USB_TO_MOSFET: track 73.6 -> 70.2 mm
- net VCC: track 274.5 -> 277.9 mm
- net USB_D+: track 51.6 -> 48.7 mm
- net BOOT: track 37.4 -> 39.7 mm
- net USB_D-: track 51.8 -> 49.8 mm
- net GNDD: track 25.4 -> 26.2 mm, vias 21 -> 65
- net Net-(J7-Pin_1): track 33.1 -> 33.9 mm
- net DRIVER_Y_nFAULT_TO_ESP32: track 68.6 -> 69.3 mm
- net DRIVER_Y_STEP_TO_ESP32: track 65.1 -> 65.8 mm
- net MODE0_TO_ESP32: track 79.6 -> 80.3 mm
- net VCC_3V3: vias 3 -> 15
- net GND: vias 71 -> 65
- added copper zone on F.Cu, net GND
- added copper zone on F.Cu, net GNDD
- added copper zone on F.Cu, net VCC_3V3
Other:
- board size 84.5 x 81.1 mm -> 92.1 x 85.4 mm
- board text added: "Fabricio Guillen Alejandro Campo"
