File: MAQUINA_DE_BRAILLE_PCB/DRIVERS.kicad_sch (KiCad schematic)
At the start: 26 parts, among them J1 Screw_Terminal_01x04, J2 Screw_Terminal_01x04, U2 DRV8825PWPR, U3 DRV8825PWPR

Commit message: last update
Parts:
- added C25, C26: 0.1uf, Capacitor_SMD:C_0805_2012Metric_Pad1.18x1.45mm_HandSolder, symbol Device:C
- R16, R17: value 0.1 -> 0.2
Connections:
- net GND: now also C25.2, C26.2
- net VCC: now also C25.1, C26.1
