File: MAQUINA_DE_BRAILLE_PCB/POWER.kicad_sch (KiCad schematic)
At the start: 24 parts, among them J3 Screw_Terminal_01x02

Commit message: last update
Parts:
- removed C5, C6: 10uF/10v, 293D106X9010A2TE3:CAP_293D-A_VSS, symbol 293D106X9010A2TE3:293D106X9010A2TE3
- added C5: 10uF/10v, 293D106X9010B2TE3:CAP_293D_B_VIS, symbol 293D106X9010B2TE3:293D106X9010B2TE3
- added C6: 10uF/10v, CAP_293D_B_VIS, symbol 293D106X9010B2TE3:293D106X9010B2TE3
Connections:
- net GND: now also C5.2, C6.2
- net MOSFET_TO_LDO: now also C5.1
- net VCC_3V3: now also C6.1
Changed lines of the file:
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@@
+	)
+	(symbol
+		(lib_id "293D106X9010B2TE3:293D106X9010B2TE3")
+		(at 137.922 39.37 270)
+		(unit 1)
+		(exclude_from_sim no)
+		(in_bom yes)
+		(on_board yes)
+		(dnp no)
+		(fields_autoplaced yes)
+		(property "Reference" "C5"
+			(at 140.97 41.9099 90)
+			(effects
+				(font
+					(size 1.524 1.524)
+				)
+				(justify left)
+			)
+		)
+		(property "Value" "10uF/10v"
+			(at 140.97 44.4499 90)
+			(effects
+				(font
+					(size 1.524 1.524)
+				)
+				(justify left)
+			)
+		)
+		(property "Footprint" "293D106X9010B2TE3:CAP_293D_B_VIS"
+			(at 137.922 39.37 0)
+			(effects
+				(font
+					(size 1.27 1.27)
+					(italic yes)
+				)
+				(hide yes)
+			)
+		)
+		(property "Datasheet" "https://www.vishay.com/doc?40002"
+			(at 137.922 39.37 0)
+			(effects
+				(font
+					(size 1.27 1.27)
+					(italic yes)
+				)
+				(hide yes)
+			)
+		)
+		(property "Description" ""
+			(at 137.922 39.37 0)
+			(effects
+				(font
+					(size 1.27 1.27)
+				)
+				(hide yes)
+			)
+		)
+		(pin "1"
+		)
+		(pin "2"
+		)
+		(instances
+			(project "MAQUINA_DE_BRAILLE"
+				(path "/9a6fa5b9-6251-4c76-8504-ded4de8e2fcc/63b065f7-e776-41e8-916c-5c22e6daf15e"
+					(reference "C5")
+					(unit 1)
+				)
+			)
+		)
+	)
+	(symbol
+		(lib_id "293D106X9010B2TE3:293D106X9010B2TE3")
+		(at 112.776 56.896 270)
+		(unit 1)
+		(exclude_from_sim no)
+		(in_bom yes)
+		(on_board yes)
+		(dnp no)
+		(fields_autoplaced yes)
+		(property "Reference" "C6"
+			(at 115.824 59.4359 90)
+			(effects
+				(font
+					(size 1.524 1.524)
+				)
+				(justify left)
+			)
+		)
+		(property "Value" "10uF/10v"
+			(at 115.824 61.9759 90)
+			(effects
+				(font
+					(size 1.524 1.524)
+				)
+				(justify left)
+			)
+		)
+		(property "Footprint" "CAP_293D_B_VIS"
+			(at 112.776 56.896 0)
+			(effects
+				(font
+					(size 1.27 1.27)
+					(italic yes)
+				)
+				(hide yes)
+			)
+		)
+		(property "Datasheet" "https://www.vishay.com/doc?40002"
+			(at 112.776 56.896 0)
+			(effects
+				(font
+					(size 1.27 1.27)
+					(italic yes)
+				)
+				(hide yes)
+			)
+		)
+		(property "Description" ""
+			(at 112.776 56.896 0)
+			(effects
+				(font
+					(size 1.27 1.27)
+				)
+				(hide yes)
+			)
+		)
+		(pin "1"
+		)
+		(pin "2"
+		)
+		(instances
+			(project ""
+				(path "/9a6fa5b9-6251-4c76-8504-ded4de8e2fcc/63b065f7-e776-41e8-916c-5c22e6daf15e"
+					(reference "C6")
+					(unit 1)
+				)
+			)
+		)
 	)
 	(symbol
@@
 	)
 	(symbol
-		(lib_id "293D106X9010A2TE3:293D106X9010A2TE3")
-		(at 137.922 39.37 270)
-		(unit 1)
-		(exclude_from_sim no)
-		(in_bom yes)
-		(on_board yes)
-		(dnp no)
-		(property "Reference" "C5"
-			(at 146.05 42.418 90)
-			(effects
-				(font
-					(size 1.524 1.524)
-				)
-				(justify right)
-			)
-		)
-		(property "Value" "10uF/10v"
-			(at 141.224 44.4499 90)
-			(effects
-				(font
-					(size 1.524 1.524)
-				)
-				(justify left)
-			)
-		)
-		(property "Footprint" "293D106X9010A2TE3:CAP_293D-A_VSS"
-			(at 137.922 39.37 0)
-			(effects
-				(font
-					(size 1.27 1.27)
-					(italic yes)
-				)
-				(hide yes)
-			)
-		)
-		(property "Datasheet" "https://www.vishay.com/doc?40002"
-			(at 137.922 39.37 0)
-			(effects
-				(font
-					(size 1.27 1.27)
-					(italic yes)
-				)
-				(hide yes)
-			)
-		)
-		(property "Description" ""
-			(at 137.922 39.37 0)
-			(effects
-				(font
-					(size 1.27 1.27)
-				)
-				(hide yes)
-			)
-		)
-		(pin "1"
-		)
-		(pin "2"
-		)
-		(instances
-			(project "MAQUINA_DE_BRAILLE"
-				(path "/9a6fa5b9-6251-4c76-8504-ded4de8e2fcc/63b065f7-e776-41e8-916c-5c22e6daf15e"
-					(reference "C5")
-					(unit 1)
-				)
-			)
-		)
-	)
-	(symbol
 		(lib_id "IHLP1616BZER4R7M11:IHLP1616BZER4R7M11")
 		(at 132.588 142.748 0)
@@
 					(unit 1)
 				)
-			)
-		)
-	)
-	(symbol
-		(lib_id "293D106X9010A2TE3:293D106X9010A2TE3")
-		(at 112.776 56.896 270)
-		(unit 1)
-		(exclude_from_sim no)
-		(in_bom yes)
-		(on_board yes)
-		(dnp no)
-		(fields_autoplaced yes)
-		(property "Reference" "C6"
-			(at 116.586 59.4359 90)
-			(effects
-				(font
-					(size 1.524 1.524)
-				)
-				(justify left)
-			)
-		)
-		(property "Value" "10uF/10v"
-			(at 116.586 61.9759 90)
-			(effects
-				(font
-					(size 1.524 1.524)
-				)
-				(justify left)
-			)
-		)
-		(property "Footprint" "293D106X9010A2TE3:CAP_293D-A_VSS"
-			(at 112.776 56.896 0)
-			(effects
-				(font
-					(size 1.27 1.27)
-					(italic yes)
-				)
-				(hide yes)
-			)
-		)
-		(property "Datasheet" "https://www.vishay.com/doc?40002"
-			(at 112.776 56.896 0)
-			(effects
-				(font
-					(size 1.27 1.27)
-					(italic yes)
-				)
-				(hide yes)
-			)
-		)
-		(property "Description" ""
-			(at 112.776 56.896 0)
-			(effects
-				(font
-					(size 1.27 1.27)
-				)
-				(hide yes)
-			)
-		)
-		(pin "1"
-		)
-		(pin "2"
-		)
-		(instances
-			(project ""
-				(path "/9a6fa5b9-6251-4c76-8504-ded4de8e2fcc/63b065f7-e776-41e8-916c-5c22e6daf15e"
-					(reference "C6")
-					(unit 1)
-				)

Commit message: last update
Parts:
- C13: value 0.1uf -> 1nf
- C14: value 6.8uf -> 6.8nf
Changed lines of the file:
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@@
 		(fields_autoplaced yes)
 		(property "Reference" "C13"
-			(at 108.458 100.8379 0)
+			(at 109.22 100.8379 0)
 			(effects
 				(font
@@
 			)
 		)
-		(property "Value" "0.1uf"
-			(at 108.458 103.3779 0)
+		(property "Value" "1nf"
+			(at 109.22 103.3779 0)
 			(effects
 				(font
@@
 			)
 		)
-		(property "Value" "6.8uf"
+		(property "Value" "6.8nf"
 			(at 178.308 121.1579 0)
 			(effects
