File: MAQUINA_DE_BRAILLE_PCB/ESP32.kicad_sch (KiCad schematic)
At the start: 20 parts, among them J4 USB_C_Receptacle_USB2.0_16P, J5 Screw_Terminal_01x03, J6 Screw_Terminal_01x03, J7 Screw_Terminal_01x02, J8 Screw_Terminal_01x16, Q1 IRLZ44NSTRLPBF, SW1 TS-1088-AR02016, SW2 TS-1088-AR02016, U1 ESP32-S3-WROOM-1-N16

Commit message: a
Parts:
- removed SW1, SW2: TS-1088-AR02016, TS-1088-AR02016:SW_TS-1088_XNP, symbol TS-1088-AR02016 -:TS-1088-AR02016
- added S1, S2: 434123025816, SW434123025816:434123025816, symbol SW434123025816:434123025816
Connections:
- net EN: now also S1.2
- net GNDD: now also S1.1, S2.1
- net at R4.1: now also S2.2
