File: MAQUINA_DE_BRAILLE_PCB/MAQUINA_DE_BRAILLE.kicad_sch (KiCad schematic)
At the start: 0 parts

Commit message: a
Parts:
- added H1, H2, H3, H4: MountingHole_Pad, MountingHole:MountingHole_3mm_Pad_Via, symbol Mechanical:MountingHole_Pad
Connections:
- new net GND: H1.1, H2.1, H3.1, H4.1
